Commit message: add week4

File: src/mbot_description/urdf/urdf/mbot_with_kinect.urdf (robot description, URDF)
Before this commit: robot mbot, 9 links, 8 joints
Links:
- removed link laser_link
- removed link second_link
- removed link stem1_link
- link base_link: geometry visual cylinder length=0.16 radius=0.20
- link left_wheel_link: geometry visual cylinder length=0.025 radius=0.06
- link right_wheel_link: geometry visual cylinder length=0.025 radius=0.06
Joints:
- removed joint laser_joint
- removed joint stem1down_joint
- removed joint stem1up_joint
- joint back_caster_joint: origin xyz=-0.15 0 -0.01 rpy=0 0 0 -> xyz=-0.18 0 -0.095 rpy=0 0 0
- joint front_caster_joint: origin xyz=0.15 0 -0.01 rpy=0 0 0 -> xyz=0.18 0 -0.095 rpy=0 0 0
- joint kinect_joint: origin xyz=0.15 0 0.04 rpy=0 0 0 -> xyz=0.15 0 0.11 rpy=0 0 0
- joint left_wheel_joint: origin xyz=0 0.178 0 rpy=0 0 0 -> xyz=0 0.19 -0.05 rpy=0 0 0
- joint right_wheel_joint: origin xyz=0 -0.178 0 rpy=0 0 0 -> xyz=0 -0.19 -0.05 rpy=0 0 0

File: src/week4_homework/urdf/urdf/mbot_base.urdf (robot description, URDF)
Before this commit: robot mbot, 6 links, 5 joints
Links:
- removed link kinect_link
Joints:
- removed joint laser_joint

File: src/week4_homework/urdf/urdf/mbot_with_camera.urdf (robot description, URDF)
Before this commit: robot mbot, 9 links, 8 joints
Links:
- removed link kinect_link
- removed link laser_link
- removed link second_link
- removed link stem1_link
- added link camera_link; visual box size=0.03 0.04 0.04
- link base_link: geometry visual cylinder length=0.16 radius=0.20
- link left_wheel_link: geometry visual cylinder length=0.025 radius=0.06
- link right_wheel_link: geometry visual cylinder length=0.025 radius=0.06
Joints:
- removed joint kinect_joint
- removed joint laser_joint
- removed joint stem1down_joint
- removed joint stem1up_joint
- added joint camera_joint: type fixed, parent base_link, child camera_link, origin xyz=0.17 0 0.10 rpy=0 0 0
- joint back_caster_joint: origin xyz=-0.15 0 -0.01 rpy=0 0 0 -> xyz=-0.18 0 -0.095 rpy=0 0 0
- joint front_caster_joint: origin xyz=0.15 0 -0.01 rpy=0 0 0 -> xyz=0.18 0 -0.095 rpy=0 0 0
- joint left_wheel_joint: origin xyz=0 0.178 0 rpy=0 0 0 -> xyz=0 0.19 -0.05 rpy=0 0 0
- joint right_wheel_joint: origin xyz=0 -0.178 0 rpy=0 0 0 -> xyz=0 -0.19 -0.05 rpy=0 0 0

File: src/week4_homework/urdf/urdf/mbot_with_laser.urdf (robot description, URDF)
Before this commit: robot mbot, 9 links, 8 joints
Links:
- removed link kinect_link
- removed link second_link
- removed link stem1_link
- link base_link: geometry visual cylinder length=0.16 radius=0.20
- link left_wheel_link: geometry visual cylinder length=0.025 radius=0.06
- link right_wheel_link: geometry visual cylinder length=0.025 radius=0.06
Joints:
- removed joint kinect_joint
- removed joint stem1down_joint
- removed joint stem1up_joint
- joint back_caster_joint: origin xyz=-0.15 0 -0.01 rpy=0 0 0 -> xyz=-0.18 0 -0.095 rpy=0 0 0
- joint front_caster_joint: origin xyz=0.15 0 -0.01 rpy=0 0 0 -> xyz=0.18 0 -0.095 rpy=0 0 0
- joint laser_joint: origin xyz=0 0 0 rpy=0 0 0 -> xyz=0 0 0.105 rpy=0 0 0; parent second_link -> base_link
- joint left_wheel_joint: origin xyz=0 0.178 0 rpy=0 0 0 -> xyz=0 0.19 -0.05 rpy=0 0 0
- joint right_wheel_joint: origin xyz=0 -0.178 0 rpy=0 0 0 -> xyz=0 -0.19 -0.05 rpy=0 0 0
