Commit message: complete mbot_base(expect stem param)

File: src/week4_homework/urdf/xacro/mbot.xacro (robot description, xacro)
@@ -1,5 +1,5 @@
 <?xml version="1.0"?>
-<robot name="arm" xmlns:xacro="http://www.ros.org/wiki/xacro">
-    <xacro:include filename="$(find mbot_description)/urdf/xacro/mbot_base.xacro" />
+<robot name="bot" xmlns:xacro="http://www.ros.org/wiki/xacro">
+    <xacro:include filename="$(find week4_homework)/urdf/xacro/mbot_base.xacro" />
     <mbot_base/>
 </robot>

File: src/week4_homework/urdf/xacro/mbot_base.xacro (robot description, xacro)
@@ -3,12 +3,12 @@
     <!-- PROPERTY LIST -->
     <xacro:property name="M_PI" value="3.1415926"/>
-    <xacro:property name="base_radius" value="0.20"/>
-    <xacro:property name="base_length" value="0.16"/>
-    <xacro:property name="wheel_radius" value="0.06"/>
-    <xacro:property name="wheel_length" value="0.025"/>
-    <xacro:property name="wheel_joint_y" value="0.19"/>
-    <xacro:property name="wheel_joint_z" value="0.05"/>
+    <xacro:property name="base_length" value="0.34"/>
+    <xacro:property name="base_height" value="0.02"/>
+    <xacro:property name="wheel_radius" value="0.04"/>
+    <xacro:property name="wheel_length" value="0.016"/>
+    <xacro:property name="wheel_joint_y" value="0.178"/>
+    <xacro:property name="wheel_joint_z" value="0"/>
     <xacro:property name="caster_radius" value="0.015"/> <!-- wheel_radius - ( base_length/2 - wheel_joint_z) -->
-    <xacro:property name="caster_joint_x" value="0.18"/>
+    <xacro:property name="caster_joint_x" value="0.15"/>
     <!-- Defining the colors used in this robot -->
     <material name="yellow">
@@ -42,5 +42,5 @@
     <xacro:macro name="caster" params="prefix reflect">
         <joint name="${prefix}_caster_joint" type="continuous">
-            <origin xyz="${reflect*caster_joint_x} 0 ${-(base_length/2 + caster_radius)}" rpy="0 0 0"/>
+            <origin xyz="${reflect*caster_joint_x} 0 ${-(base_height/2 + caster_radius)}" rpy="0 0 0"/>
             <parent link="base_link"/>
             <child link="${prefix}_caster_link"/>
@@ -67,5 +67,5 @@
         </link>
         <joint name="base_footprint_joint" type="fixed">
-            <origin xyz="0 0 ${base_length/2 + caster_radius*2}" rpy="0 0 0" />
+            <origin xyz="0 0 ${base_height/2 + caster_radius*2}" rpy="0 0 0" />
             <parent link="base_footprint"/>
             <child link="base_link" />
@@ -75,9 +75,39 @@
                 <origin xyz=" 0 0 0" rpy="0 0 0" />
                 <geometry>
-                    <cylinder length="${base_length}" radius="${base_radius}"/>
+                    <box size="${base_length} ${base_length} ${base_height}"/>
                 </geometry>
                 <material name="yellow" />
             </visual>
         </link>
+          <joint name="stem1down_joint" type="fixed">
+        <origin xyz="0 0 0.01" rpy="0 0 0"/>
+        <parent link="base_link"/>
+        <child link="stem1_link"/>
+    </joint>
+    <link name="stem1_link">
+        <visual>
+            <origin xyz=" 0 0 0.05" rpy="0 0 0" />
+            <geometry>
+                <cylinder length="0.1" radius="0.015"/>
+            </geometry>
+            <material name="yellow">
+            </material>
+        </visual>
+    </link>
+    <joint name="stem1up_joint" type="fixed">
+        <origin xyz="0 0 0.09" rpy="0 0 0"/>
+        <parent link="stem1_link"/>
+        <child link="second_link"/>
+    </joint>
+        <link name="second_link">
+        <visual>
+            <origin xyz="0 0 0" rpy="0 0 0" />
+            <geometry>
+                <box size="${base_length} ${base_length} ${base_height}"/>
+            </geometry>
+            <material name="yellow">
+            </material>
+        </visual>
+    </link>
         <wheel prefix="left" reflect="-1"/>
         <wheel prefix="right" reflect="1"/>
