Commit message: complete week4 t3

File: src/week4_homework/urdf/xacro/gazebo/mbot_kinect_lidar_gazebo.xacro (robot description, xacro)
@@ -1,7 +1,7 @@
 <?xml version="1.0"?>
 <robot name="arm" xmlns:xacro="http://www.ros.org/wiki/xacro">
-    <xacro:include filename="$(find week4_homework)/urdf/xacro/mbot_base_gazebo.xacro" />
-    <xacro:include filename="$(find week4_homework)/urdf/xacro/sensors/kinect_gazebo.xacro" />
-    <xacro:include filename="$(find week4_homework)/urdf/xacro/sensors/lidar_gazebo.xacro" />
+    <xacro:include filename="$(find mbot_description)/urdf/xacro/gazebo/mbot_base_gazebo.xacro" />
+    <xacro:include filename="$(find mbot_description)/urdf/xacro/sensors/lidar_gazebo.xacro" />
+    <xacro:include filename="$(find mbot_description)/urdf/xacro/sensors/kinect_gazebo.xacro" />
     <xacro:property name="kinect_offset_x" value="0.15" />
     <xacro:property name="kinect_offset_y" value="0" />
@@ -10,6 +10,4 @@
     <xacro:property name="lidar_offset_y" value="0" />
     <xacro:property name="lidar_offset_z" value="0.025" />
-    <mbot_base/>
-    <!-- Camera -->
     <joint name="kinect_joint" type="fixed">
         <origin xyz="${kinect_offset_x} ${kinect_offset_y} ${kinect_offset_z}" rpy="0 0 0" />
@@ -21,6 +19,7 @@
         <origin xyz="${lidar_offset_x} ${lidar_offset_y} ${lidar_offset_z}" rpy="0 0 0" />
         <parent link="second_link"/>
-        <child link="lidar_link"/>
+        <child link="laser_link"/>
     </joint>
-    <xacro:rplidar prefix="lidar"/>
+    <xacro:rplidar prefix="laser"/>
+    <mbot_base_gazebo/>
 </robot>
