Commit message: dsaf

File: src/week3_homework/urdf/mbot_base.urdf (robot description, URDF)
Before this commit: robot mbot, 5 links, 4 joints
Links:
- removed link back_caster_link
- removed link front_caster_link
- removed link left_wheel_link
- removed link right_wheel_link
Joints:
- removed joint back_caster_joint
- removed joint front_caster_joint
- removed joint left_wheel_joint
- removed joint right_wheel_joint

Commit message: o

File: src/week3_homework/urdf/mbot_base.urdf (robot description, URDF)
Before this commit: robot mbot, 1 links, 0 joints
Links:
- added link back_caster_link; visual sphere radius=0.015
- added link front_caster_link; visual sphere radius=0.015
- added link left_wheel_link; visual cylinder length=0.025 radius=0.06
- added link right_wheel_link; visual cylinder length=0.025 radius=0.06
Joints:
- added joint back_caster_joint: type continuous, parent base_link, child back_caster_link, origin xyz=-0.18 0 -0.095 rpy=0 0 0, axis 0 1 0
- added joint front_caster_joint: type continuous, parent base_link, child front_caster_link, origin xyz=0.18 0 -0.095 rpy=0 0 0, axis 0 1 0
- added joint left_wheel_joint: type continuous, parent base_link, child left_wheel_link, origin xyz=0 0.19 -0.05 rpy=0 0 0, axis 0 1 0
- added joint right_wheel_joint: type continuous, parent base_link, child right_wheel_link, origin xyz=0 -0.19 -0.05 rpy=0 0 0, axis 0 1 0

Commit message: ';

File: src/week3_homework/urdf/mbot_base.urdf (robot description, URDF)
Before this commit: robot mbot, 5 links, 4 joints
Links:
- link base_link: geometry visual box size=0.34 0.34 0.02
- link left_wheel_link: geometry visual cylinder length=0.016 radius=0.04
- link right_wheel_link: geometry visual cylinder length=0.016 radius=0.04
Joints:
- joint back_caster_joint: origin xyz=-0.18 0 -0.095 rpy=0 0 0 -> xyz=-0.15 0 -0.01 rpy=0 0 0
- joint front_caster_joint: origin xyz=0.18 0 -0.095 rpy=0 0 0 -> xyz=0.15 0 -0.01 rpy=0 0 0
- joint left_wheel_joint: origin xyz=0 0.19 -0.05 rpy=0 0 0 -> xyz=0 0.178 0 rpy=0 0 0
- joint right_wheel_joint: origin xyz=0 -0.19 -0.05 rpy=0 0 0 -> xyz=0 -0.178 0 rpy=0 0 0

Commit message: add kinect

File: src/week3_homework/urdf/mbot_base.urdf (robot description, URDF)
Before this commit: robot mbot, 5 links, 4 joints
Links:
- added link kinect_link; visual mesh filename=package://mbot_description/meshes/kinect.dae
- added link second_link; visual box size=0.34 0.34 0.02
- added link stem1_link; visual cylinder length=0.28 radius=0.02
- added link stem2_link; visual cylinder length=0.28 radius=0.02
Joints:
- added joint kinect_joint: type fixed, parent base_link, child kinect_link, origin xyz=0.15 0 0.04 rpy=0 0 0
- added joint stem1down_joint: type fixed, parent base_link, child stem1_link, origin xyz=0 0.19 -0.05 rpy=0 0 0
- added joint stem1up_joint: type fixed, parent stem1_link, child second_link, origin xyz=0 0.19 -0.05 rpy=0 0 0
- added joint stem2down_joint: type fixed, parent base_link, child stem2_link, origin xyz=0 0.19 -0.05 rpy=0 0 0
- added joint stem2up_joint: type fixed, parent stem2_link, child second_link, origin xyz=0 0.19 -0.05 rpy=0 0 0

Commit message: solve caster postion

File: src/week3_homework/urdf/mbot_base.urdf (robot description, URDF)
Before this commit: robot mbot, 9 links, 8 joints
Joints:
- joint back_caster_joint: origin xyz=-0.15 0 -0.01 rpy=0 0 0 -> xyz=-0.15 0 -0.025 rpy=0 0 0
- joint front_caster_joint: origin xyz=0.15 0 -0.01 rpy=0 0 0 -> xyz=0.15 0 -0.025 rpy=0 0 0

Commit message: delete mbotdesc and change some question without mbot desc  test all homework and take a screenshot

File: src/week3_homework/urdf/mbot_base.urdf (robot description, URDF)
Before this commit: robot mbot, 9 links, 8 joints
Links:
- link kinect_link: geometry visual mesh filename=package://week4_homework/meshes/kinect.dae

File: src/week4_homework/urdf/xacro/gazebo/mbot_kinect_lidar_gazebo.xacro (robot description, xacro)
@@ -1,7 +1,7 @@
 <?xml version="1.0"?>
 <robot name="arm" xmlns:xacro="http://www.ros.org/wiki/xacro">
-    <xacro:include filename="$(find mbot_description)/urdf/xacro/gazebo/mbot_base_gazebo.xacro" />
-    <xacro:include filename="$(find mbot_description)/urdf/xacro/sensors/lidar_gazebo.xacro" />
-    <xacro:include filename="$(find mbot_description)/urdf/xacro/sensors/kinect_gazebo.xacro" />
+    <xacro:include filename="$(find week4_homework)/urdf/xacro/gazebo/mbot_base_gazebo.xacro" />
+    <xacro:include filename="$(find week4_homework)/urdf/xacro/sensors/lidar_gazebo.xacro" />
+    <xacro:include filename="$(find week4_homework)/urdf/xacro/sensors/kinect_gazebo.xacro" />
     <xacro:property name="kinect_offset_x" value="0.15" />
     <xacro:property name="kinect_offset_y" value="0" />

File: src/week4_homework/urdf/xacro/sensors/kinect.xacro (robot description, xacro)
@@ -7,5 +7,5 @@
                 <origin xyz="0 0 0" rpy="0 0 ${M_PI/2}"/>
                 <geometry>
-                    <mesh filename="package://mbot_description/meshes/kinect.dae" />
+                    <mesh filename="package://week4_homework/meshes/kinect.dae" />
                 </geometry>
             </visual>

File: src/week4_homework/urdf/xacro/sensors/kinect_gazebo.xacro (robot description, xacro)
@@ -9,5 +9,5 @@
                 <origin xyz="0 0 0" rpy="0 0 ${M_PI/2}"/>
                 <geometry>
-                    <mesh filename="package://mbot_description/meshes/kinect.dae" />
+                    <mesh filename="package://week4_homework/meshes/kinect.dae" />
                 </geometry>
             </visual>
